File: imacro.kicad_pcb (KiCad board)
At the start: 2 copper layers, 57.2 x 95.2 mm, 29 parts, among them SW0:0 Choc, SW0:1 Choc, SW0:2 Choc, SW1 TOGGLE, SW1:0 Choc, SW1:1 Choc, SW1:2 Choc, SW2:0 Choc, SW2:1 Choc, SW2:2 Choc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

Commit message: adjust mask clearance to OSH Park spec
Other:
- rule pad_to_mask_clearance: 0.2 -> 0.0508
Changed lines of the file:
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@@
     (pad_size 1.524 1.524)
     (pad_drill 0.762)
-    (pad_to_mask_clearance 0.2)
+    (pad_to_mask_clearance 0.0508)
     (aux_axis_origin 0 0)
     (visible_elements FFFFFF7F)

Commit message: Don’t use pin 9 on the feather so it can be used to read the battery level
Connections:
- U1 pad 19: Net-(U1-Pad19) -> /ROW3
- U1 pad 8: /ROW3 -> Net-(U1-Pad8)
Routing:
- net /ROW3: track 63.3 -> 43.9 mm
Changed lines of the file:
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@@
-(kicad_pcb (version 4) (host pcbnew 4.0.7-e2-6376~58~ubuntu16.04.1)
+(kicad_pcb (version 4) (host pcbnew 4.0.7)
   (general
     (links 41)
@@
     (thickness 1.6)
     (drawings 11)
-    (tracks 155)
+    (tracks 154)
     (zones 0)
     (modules 29)
@@
   (net 31 "Net-(U1-Pad17)")
   (net 32 "Net-(U1-Pad18)")
-  (net 33 "Net-(U1-Pad19)")
-  (net 34 "Net-(U1-Pad20)")
-  (net 35 "Net-(U1-Pad21)")
-  (net 36 "Net-(U1-Pad22)")
-  (net 37 "Net-(U1-Pad23)")
-  (net 38 "Net-(U1-Pad24)")
-  (net 39 "Net-(U1-Pad26)")
-  (net 40 "Net-(U1-Pad27)")
-  (net 41 "Net-(U1-Pad28)")
+  (net 33 "Net-(U1-Pad20)")
+  (net 34 "Net-(U1-Pad21)")
+  (net 35 "Net-(U1-Pad22)")
+  (net 36 "Net-(U1-Pad23)")
+  (net 37 "Net-(U1-Pad24)")
+  (net 38 "Net-(U1-Pad26)")
+  (net 39 "Net-(U1-Pad27)")
+  (net 40 "Net-(U1-Pad28)")
+  (net 41 "Net-(U1-Pad8)")
   (net_class Default "This is the default net class."
     (clearance 0.254)
@@
     (add_net "Net-(U1-Pad17)")
     (add_net "Net-(U1-Pad18)")
-    (add_net "Net-(U1-Pad19)")
     (add_net "Net-(U1-Pad20)")
     (add_net "Net-(U1-Pad21)")
@@
     (add_net "Net-(U1-Pad28)")
     (add_net "Net-(U1-Pad4)")
+    (add_net "Net-(U1-Pad8)")
   )
   (module imacro:GPTS_SPST_Pushbutton (layer B.Cu)
@@
       (net 21 /ROW2))
     (pad 8 thru_hole circle (at 8.89 10.16 180) (size 1.524 1.524) (drill 1.02) (layers *.Cu *.Mask)
-      (net 22 /ROW3))
+      (net 41 "Net-(U1-Pad8)"))
     (pad 9 thru_hole circle (at 11.43 10.16 180) (size 1.524 1.524) (drill 1.02) (layers *.Cu *.Mask)
       (net 1 /COL0))
@@
       (net 32 "Net-(U1-Pad18)"))
     (pad 19 thru_hole circle (at 3.81 -10.16 180) (size 1.524 1.524) (drill 1.02) (layers *.Cu *.Mask)
-      (net 33 "Net-(U1-Pad19)"))
+      (net 22 /ROW3))
     (pad 20 thru_hole circle (at 1.27 -10.16 180) (size 1.524 1.524) (drill 1.02) (layers *.Cu *.Mask)
-      (net 34 "Net-(U1-Pad20)"))
+      (net 33 "Net-(U1-Pad20)"))
     (pad 21 thru_hole circle (at -1.27 -10.16 180) (size 1.524 1.524) (drill 1.02) (layers *.Cu *.Mask)
-      (net 35 "Net-(U1-Pad21)"))
+      (net 34 "Net-(U1-Pad21)"))
     (pad 22 thru_hole circle (at -3.81 -10.16 180) (size 1.524 1.524) (drill 1.02) (layers *.Cu *.Mask)
-      (net 36 "Net-(U1-Pad22)"))
+      (net 35 "Net-(U1-Pad22)"))
     (pad 23 thru_hole circle (at -6.35 -10.16 180) (size 1.524 1.524) (drill 1.02) (layers *.Cu *.Mask)
-      (net 37 "Net-(U1-Pad23)"))
+      (net 36 "Net-(U1-Pad23)"))
     (pad 24 thru_hole circle (at -8.89 -10.16 180) (size 1.524 1.524) (drill 1.02) (layers *.Cu *.Mask)
-      (net 38 "Net-(U1-Pad24)"))
+      (net 37 "Net-(U1-Pad24)"))
     (pad 25 thru_hole circle (at -11.43 -10.16 180) (size 1.524 1.524) (drill 1.02) (layers *.Cu *.Mask)
       (net 18 GND))
     (pad 26 thru_hole circle (at -13.97 -10.16 180) (size 1.524 1.524) (drill 1.02) (layers *.Cu *.Mask)
-      (net 39 "Net-(U1-Pad26)"))
+      (net 38 "Net-(U1-Pad26)"))
     (pad 27 thru_hole circle (at -16.51 -10.16 180) (size 1.524 1.524) (drill 1.02) (layers *.Cu *.Mask)
-      (net 40 "Net-(U1-Pad27)"))
+      (net 39 "Net-(U1-Pad27)"))
     (pad 28 thru_hole circle (at -19.05 -10.16 180) (size 1.524 1.524) (drill 1.02) (layers *.Cu *.Mask)
-      (net 41 "Net-(U1-Pad28)"))
+      (net 40 "Net-(U1-Pad28)"))
   )
   (module imacro:PG1350 (layer F.Cu)
@@
   (segment (start 100.0125 94.00625) (end 119.0625 94.00625) (width 0.25) (layer F.Cu) (net 21))
   (segment (start 80.9625 94.00625) (end 100.0125 94.00625) (width 0.25) (layer F.Cu) (net 21))
-  (segment (start 91.1225 54.13375) (end 91.1225 68.42125) (width 0.25) (layer B.Cu) (net 22))
-  (segment (start 89.35 70.19375) (end 80.9625 70.19375) (width 0.25) (layer B.Cu) (net 22))
-  (segment (start 91.1225 68.42125) (end 89.35 70.19375) (width 0.25) (layer B.Cu) (net 22))
+  (segment (start 96.2025 74.45375) (end 96.2025 74.00375) (width 0.254) (layer F.Cu) (net 22) (status C00000))
+  (segment (start 96.2025 74.00375) (end 100.0125 70.19375) (width 0.254) (layer F.Cu) (net 22) (status C00000))
   (segment (start 80.9625 70.19375) (end 100.0125 70.19375) (width 0.25) (layer F.Cu) (net 22))
   (segment (start 119.0625 70.19375) (end 100.0125 70.19375) (width 0.25) (layer F.Cu) (net 22))

Commit message: accomodate smaller case; rotate Feather board around for new battery cable position; improve trace routing somewhat
Parts:
- removed the REF*** at (77.5, 46.0)
- added REF***: OSHW-Logo_7.5x8mm_Copper, Symbols:OSHW-Logo_7.5x8mm_Copper, F.Cu at (90.5, 99.0)
- moved SW1 77.0 mm to (78.0, 123.0), turned to 0 degrees
- moved D1 18.8 mm to (125.5, 111.5)
- moved QI1 18.5 mm to (123.5, 116.5), turned to 180 degrees
- moved U1 0.21 mm to (100.0, 64.5), turned to 0 degrees
Connections:
- U1 pad 14: /COL1 -> /COL2
- U1 pad 15: /COL2 -> /COL1
Routing:
- net /5V_USB: track 129.3 -> 70.0 mm
- net /ROW2: track 103.0 -> 60.4 mm
- net /COL1: track 66.1 -> 106.9 mm, vias 0 -> 4
- net /ROW1: track 124.4 -> 94.2 mm
- net /ROW0: track 144.4 -> 118.4 mm
- net Net-(SW1-Pad2): track 33.7 -> 52.1 mm, vias 1 -> 2
- net /ROW3: track 43.9 -> 56.4 mm
- net /COL2: track 81.5 -> 73.6 mm
- net /COL0: track 77.8 -> 75.9 mm
- net Net-(D1-Pad2): track 4.52 -> 3.95 mm
Other:
- board size 57.2 x 95.2 mm -> 57.2 x 83.3 mm
- net class Power added: clearance 0.254, trace_width 0.508, via_dia 0.6858, via_drill 0.3302

Commit message: Move D0:0 for power button clearance
Parts:
- moved D0:0 11.1 mm to (88.0, 130.0)
Routing:
- net /COL0: track 75.9 -> 88.3 mm
Changed lines of the file:
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@@
     (thickness 1.6)
     (drawings 9)
-    (tracks 154)
+    (tracks 155)
     (zones 0)
     (modules 29)
@@
   )
   (module Diodes_SMD:D_SOD-123 (layer B.Cu)
-    (at 80.9625 121.44375 180)
+    (at 88 130 180)
     (descr SOD-123)
     (tags SOD-123)
@@
   (gr_line (start 128.5875 52.3875) (end 128.5875 135.73125) (angle 90) (layer Edge.Cuts) (width 0.15))
   (gr_line (start 71.4375 135.73125) (end 71.4375 52.3875) (angle 90) (layer Edge.Cuts) (width 0.15))
+  (segment (start 84 103.78125) (end 82.6125 102.39375) (width 0.254) (layer B.Cu) (net 1))
+  (segment (start 84 127) (end 84 103.78125) (width 0.254) (layer B.Cu) (net 1))
+  (segment (start 85 128) (end 84 127) (width 0.254) (layer B.Cu) (net 1))
+  (segment (start 87 128) (end 85 128) (width 0.254) (layer B.Cu) (net 1))
+  (segment (start 89 130) (end 87 128) (width 0.254) (layer B.Cu) (net 1))
+  (segment (start 89.65 130) (end 89 130) (width 0.254) (layer B.Cu) (net 1))
   (segment (start 111.43 74.66) (end 111.43 78.57) (width 0.254) (layer B.Cu) (net 1))
   (segment (start 109.0375 80.9625) (end 82.6125 80.9625) (width 0.254) (layer B.Cu) (net 1))
@@
   (segment (start 83.34375 95.25) (end 83.34375 84.075) (width 0.25) (layer B.Cu) (net 1))
   (segment (start 82.6125 95.98125) (end 83.34375 95.25) (width 0.25) (layer B.Cu) (net 1))
-  (segment (start 82.6125 121.44375) (end 82.6125 115.03125) (width 0.25) (layer B.Cu) (net 1))
-  (segment (start 83.34375 103.125) (end 82.6125 102.39375) (width 0.25) (layer B.Cu) (net 1))
-  (segment (start 83.34375 114.3) (end 83.34375 103.125) (width 0.25) (layer B.Cu) (net 1))
-  (segment (start 82.6125 115.03125) (end 83.34375 114.3) (width 0.25) (layer B.Cu) (net 1))
-  (segment (start 75.9625 130.00625) (end 77.1625 130.00625) (width 0.25) (layer B.Cu) (net 2))
-  (segment (start 78.58125 122.175) (end 79.3125 121.44375) (width 0.25) (layer B.Cu) (net 2))
-  (segment (start 78.58125 128.5875) (end 78.58125 122.175) (width 0.25) (layer B.Cu) (net 2))
-  (segment (start 77.1625 130.00625) (end 78.58125 128.5875) (width 0.25) (layer B.Cu) (net 2))
+  (segment (start 75.9625 130.00625) (end 86.34375 130.00625) (width 0.254) (layer B.Cu) (net 2))
+  (segment (start 86.34375 130.00625) (end 86.35 130) (width 0.254) (layer B.Cu) (net 2))
+  (segment (start 86.65 130) (end 86.65 129.65) (width 0.254) (layer B.Cu) (net 2))
   (segment (start 82.6125 78.58125) (end 82.6125 71.8875) (width 0.254) (layer B.Cu) (net 3))
   (segment (start 110.5 58) (end 113.97 54.53) (width 0.254) (layer B.Cu) (net 3))
