File: PCB/imacro.sch (KiCad schematic (older format))
At the start: 28 parts, among them SW0:0 Choc, SW0:1 Choc, SW0:2 Choc, SW1 TOGGLE, SW1:0 Choc, SW1:1 Choc, SW1:2 Choc, SW2:0 Choc, SW2:1 Choc, SW2:2 Choc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

Commit message: Improve switch footprints (requires daprice/keyswitches.pretty ); increase annular ring size on other footprints; add positive indicator to Qi charger connection
Parts:
- SW0:0, SW0:1, SW0:2, SW1:0, SW1:1, SW1:2, SW2:0, SW2:1, SW2:2, SW3:0, SW3:1, SW3:2: footprint imacro:PG1350 -> keyswitches:PG1350
Changed lines of the file:
@@
 F 0 "SW3:0" H 6200 2200 50  0000 L CNN
 F 1 "Choc" H 6150 2040 50  0000 C CNN
-F 2 "imacro:PG1350" H 6150 2300 50  0001 C CNN
+F 2 "keyswitches:PG1350" H 6150 2300 50  0001 C CNN
 F 3 "" H 6150 2300 50  0001 C CNN
 	1    6150 2100
@@
 F 0 "SW3:1" H 6900 2200 50  0000 L CNN
 F 1 "Choc" H 6850 2040 50  0000 C CNN
-F 2 "imacro:PG1350" H 6850 2300 50  0001 C CNN
+F 2 "keyswitches:PG1350" H 6850 2300 50  0001 C CNN
 F 3 "" H 6850 2300 50  0001 C CNN
 	1    6850 2100
@@
 F 0 "SW3:2" H 7600 2200 50  0000 L CNN
 F 1 "Choc" H 7550 2040 50  0000 C CNN
-F 2 "imacro:PG1350" H 7550 2300 50  0001 C CNN
+F 2 "keyswitches:PG1350" H 7550 2300 50  0001 C CNN
 F 3 "" H 7550 2300 50  0001 C CNN
 	1    7550 2100
@@
 F 0 "SW2:0" H 6200 2900 50  0000 L CNN
 F 1 "Choc" H 6150 2740 50  0000 C CNN
-F 2 "imacro:PG1350" H 6150 3000 50  0001 C CNN
+F 2 "keyswitches:PG1350" H 6150 3000 50  0001 C CNN
 F 3 "" H 6150 3000 50  0001 C CNN
 	1    6150 2800
@@
 F 0 "SW2:1" H 6900 2900 50  0000 L CNN
 F 1 "Choc" H 6850 2740 50  0000 C CNN
-F 2 "imacro:PG1350" H 6850 3000 50  0001 C CNN
+F 2 "keyswitches:PG1350" H 6850 3000 50  0001 C CNN
 F 3 "" H 6850 3000 50  0001 C CNN
 	1    6850 2800
@@
 F 0 "SW2:2" H 7600 2900 50  0000 L CNN
 F 1 "Choc" H 7550 2740 50  0000 C CNN
-F 2 "imacro:PG1350" H 7550 3000 50  0001 C CNN
+F 2 "keyswitches:PG1350" H 7550 3000 50  0001 C CNN
 F 3 "" H 7550 3000 50  0001 C CNN
 	1    7550 2800
@@
 F 0 "SW1:0" H 6200 3600 50  0000 L CNN
 F 1 "Choc" H 6150 3440 50  0000 C CNN
-F 2 "imacro:PG1350" H 6150 3700 50  0001 C CNN
+F 2 "keyswitches:PG1350" H 6150 3700 50  0001 C CNN
 F 3 "" H 6150 3700 50  0001 C CNN
 	1    6150 3500
@@
 F 0 "SW1:1" H 6900 3600 50  0000 L CNN
 F 1 "Choc" H 6850 3440 50  0000 C CNN
-F 2 "imacro:PG1350" H 6850 3700 50  0001 C CNN
+F 2 "keyswitches:PG1350" H 6850 3700 50  0001 C CNN
 F 3 "" H 6850 3700 50  0001 C CNN
 	1    6850 3500
@@
 F 0 "SW1:2" H 7600 3600 50  0000 L CNN
 F 1 "Choc" H 7550 3440 50  0000 C CNN
-F 2 "imacro:PG1350" H 7550 3700 50  0001 C CNN
+F 2 "keyswitches:PG1350" H 7550 3700 50  0001 C CNN
 F 3 "" H 7550 3700 50  0001 C CNN
 	1    7550 3500
@@
 F 0 "SW0:0" H 6200 4300 50  0000 L CNN
 F 1 "Choc" H 6150 4140 50  0000 C CNN
-F 2 "imacro:PG1350" H 6150 4400 50  0001 C CNN
+F 2 "keyswitches:PG1350" H 6150 4400 50  0001 C CNN
 F 3 "" H 6150 4400 50  0001 C CNN
 	1    6150 4200
@@
 F 0 "SW0:1" H 6900 4300 50  0000 L CNN
 F 1 "Choc" H 6850 4140 50  0000 C CNN
-F 2 "imacro:PG1350" H 6850 4400 50  0001 C CNN
+F 2 "keyswitches:PG1350" H 6850 4400 50  0001 C CNN
 F 3 "" H 6850 4400 50  0001 C CNN
 	1    6850 4200
@@
 F 0 "SW0:2" H 7600 4300 50  0000 L CNN
 F 1 "Choc" H 7550 4140 50  0000 C CNN
-F 2 "imacro:PG1350" H 7550 4400 50  0001 C CNN
+F 2 "keyswitches:PG1350" H 7550 4400 50  0001 C CNN
 F 3 "" H 7550 4400 50  0001 C CNN
 	1    7550 4200
